Commit message: Robot Sensors

File: my_robot/urdf/my_robot.xacro (robot description, xacro)
@@ -1,57 +1,261 @@
 <?xml version='1.0'?>
 <robot name="my_robot" xmlns:xacro="http://www.ros.org/wiki/xacro">
-  <link name="robot_footprint"></link>
-  <joint name="robot_footprint_joint" type="fixed">
-    <origin xyz="0 0 0" rpy="0 0 0" />
-    <parent link="robot_footprint"/>
-    <child link="chassis" />
-  </joint>
-  <link name='chassis'>
-    <pose>0 0 0.1 0 0 0</pose>
-    <inertial>
-      <mass value="15.0"/>
-      <origin xyz="0.0 0 0" rpy=" 0 0 0"/>
-      <inertia
-          ixx="0.1" ixy="0" ixz="0"
-          iyy="0.1" iyz="0"
-          izz="0.1"
-      />
-    </inertial>
-    <collision name='collision'>
-      <origin xyz="0 0 0" rpy=" 0 0 0"/>
-      <geometry>
-        <box size=".4 .2 .1"/>
-      </geometry>
-    </collision>
-    <visual name='chassis_visual'>
-      <origin xyz="0 0 0" rpy=" 0 0 0"/>
-      <geometry>
-        <box size=".4 .2 .1"/>
-      </geometry>
-    </visual>
-    <collision name='back_caster_collision'>
-      <origin xyz="-0.15 0 -0.05" rpy=" 0 0 0"/>
-      <geometry>
-        <sphere radius="0.0499"/>
-      </geometry>
-    </collision>
-    <visual name='back_caster_visual'>
-      <origin xyz="-0.15 0 -0.05" rpy=" 0 0 0"/>
-      <geometry>
-        <sphere radius="0.05"/>
-      </geometry>
-    </visual>
-    <collision name='front_caster_collision'>
-      <origin xyz="0.15 0 -0.05" rpy=" 0 0 0"/>
-      <geometry>
-        <sphere radius="0.0499"/>
-      </geometry>
-    </collision>
-    <visual name='front_caster_visual'>
-      <origin xyz="0.15 0 -0.05" rpy=" 0 0 0"/>
-      <geometry>
-        <sphere radius="0.05"/>
-      </geometry>
-    </visual>
-  </link>
+    <link name="robot_footprint"></link>
+    <link name="crossbar_main">
+        <pose>0 0 0.1 0 0 0</pose>
+        <inertial>
+            <mass value="1.0"/>
+            <origin xyz="0.0 0 0" rpy=" 0 0 0"/>
+            <inertia
+                ixx="0.1" ixy="0" ixz="0"
+                iyy="0.1" iyz="0"
+                izz="0.1"
+            />
+        </inertial>
+        <collision name='crossbar_main_collision'>
+            <origin xyz="0 0 0" rpy=" 0 0 0"/>
+            <geometry>
+                <box size="0.1 0.5 0.05"/>
+            </geometry>
+        </collision>
+        <visual name='crossbar_main_visual'>
+            <origin xyz="0 0 0" rpy=" 0 0 0"/>
+            <geometry>
+                <box size="0.1 0.5 0.05"/>
+            </geometry>
+        </visual>
+        <collision name='caster_collision'>
+            <origin xyz="0 -0.25 -0.05" rpy=" 0 0 0"/>
+            <geometry>
+                <sphere radius="0.05"/>
+            </geometry>
+        </collision>
+        <visual name='caster_visual'>
+            <origin xyz="0 -0.25 -0.05" rpy=" 0 0 0"/>
+            <geometry>
+                <sphere radius="0.05"/>
+            </geometry>
+        </visual>
+    </link>
+    <link name="crossbar_trans_forward">
+        <pose>0 0 0.1 0 0 0</pose>
+        <inertial>
+            <mass value="0.5"/>
+            <origin xyz="0.0 0 0" rpy=" 0 0 0"/>
+            <inertia
+                ixx="0.1" ixy="0" ixz="0"
+                iyy="0.1" iyz="0"
+                izz="0.1"
+            />
+        </inertial>
+        <collision name='crossbar_trans_forward_collision'>
+            <origin xyz="0 0 0" rpy=" 0 0 0"/>
+            <geometry>
+                <box size="0.5 0.05 0.05"/>
+            </geometry>
+        </collision>
+        <visual name='crossbar_trans_forward_visual'>
+            <origin xyz="0 0 0" rpy=" 0 0 0"/>
+            <geometry>
+                <box size="0.5 0.05 0.05"/>
+            </geometry>
+        </visual>
+    </link>
+    <link name="crossbar_trans_center">
+        <pose>0 0 0.1 0 0 0</pose>
+        <inertial>
+            <mass value="0.5"/>
+            <origin xyz="0.0 0 0" rpy=" 0 0 0"/>
+            <inertia
+                ixx="0.1" ixy="0" ixz="0"
+                iyy="0.1" iyz="0"
+                izz="0.1"
+            />
+        </inertial>
+        <collision name='crossbar_trans_center_collision'>
+            <origin xyz="0 0 0" rpy=" 0 0 0"/>
+            <geometry>
+                <box size="0.4 0.05 0.05"/>
+            </geometry>
+        </collision>
+        <visual name='crossbar_trans_center_visual'>
+            <origin xyz="0 0 0" rpy=" 0 0 0"/>
+            <geometry>
+                <box size="0.4 0.05 0.05"/>
+            </geometry>
+        </visual>
+    </link>
+    <link name="tail">
+        <pose>0 0 0.1 0 0 0</pose>
+        <inertial>
+            <mass value="0.5"/>
+            <origin xyz="0.0 0 0" rpy=" 0 0 0"/>
+            <inertia
+                ixx="0.1" ixy="0" ixz="0"
+                iyy="0.1" iyz="0"
+                izz="0.1"
+            />
+        </inertial>
+        <collision name='tail_collision'>
+            <origin xyz="0 0 0" rpy=" 0 0 0"/>
+            <geometry>
+                <cylinder radius="0.15" length="0.15"/>
+            </geometry>
+        </collision>
+        <visual name='tail_visual'>
+            <origin xyz="0 0 0" rpy=" 0 0 0"/>
+            <geometry>
+                <cylinder radius="0.15" length="0.15"/>
+            </geometry>
+        </visual>
+    </link>
+    <link name="left_wheel">
+        <pose>0 0 0.1 0 0 0</pose>
+        <collision>
+            <geometry>
+                <cylinder radius="0.1" length="0.05"/>
+            </geometry>
+            <origin xyz="0 0 0" rpy="0 1.5707 0"/>
+        </collision>
+        <inertial>
+            <origin xyz="0 0 0" rpy="0 1.5707 0"/>
+            <mass value="0.1"/>
+            <inertia ixx="0.1" ixy="0" ixz="0"  iyy="0.1" iyz="0" izz="0.1"/>
+        </inertial>
+        <visual>
+            <geometry>
+                <cylinder radius="0.1" length="0.05"/>
+            </geometry>
+            <origin xyz="0 0 0" rpy="0 1.5707 0"/>
+        </visual>
+    </link>
+    <link name="right_wheel">
+        <pose>0 0 0.1 0 0 0</pose>
+        <collision>
+            <geometry>
+                <cylinder radius="0.1" length="0.05"/>
+            </geometry>
+            <origin xyz="0 0 0" rpy="0 1.5707 0"/>
+        </collision>
+        <inertial>
+            <origin xyz="0 0 0" rpy="0 1.5707 0"/>
+            <mass value="0.1"/>
+            <inertia ixx="0.1" ixy="0" ixz="0"  iyy="0.1" iyz="0" izz="0.1"/>
+        </inertial>
+        <visual>
+            <geometry>
+                <cylinder radius="0.1" length="0.05"/>
+            </geometry>
+            <origin xyz="0 0 0" rpy="0 1.5707 0"/>
+        </visual>
+    </link>
+    <link name="camera">
+        <inertial>
+        <mass value="0.1"/>
+        <origin xyz="0 0 0" rpy="0 0 0"/>
+        <box_inertia sizeX="0.05" sizeY="0.05" sizeZ="0.05" mass="0.1"/>
+        <inertia ixx="1e-6" ixy="0" ixz="0" iyy="1e-6" iyz="0" izz="1e-6"/>
+        </inertial>
+        <collision>
+        <origin xyz="0 0 0" rpy="1.5707 0 0"/>
+        <geometry>
+            <cylinder radius="0.025" length="0.05"/>
+        </geometry>
+        </collision>
+        <visual>
+        <origin xyz="0 0 0" rpy="1.5707 0 0"/>
+        <geometry>
+            <cylinder radius="0.025" length="0.05"/>
+        </geometry>
+        </visual>
+    </link>
+    <link name="hokuyo">
+        <inertial>
+        <mass value="1e-1"/>
+        <origin xyz="0 0 0" rpy="0 0 0"/>
+        <box_inertia sizeX="0.05" sizeY="0.05" sizeZ="0.05" mass="0.1"/>
+        <inertia ixx="1e-6" ixy="0" ixz="0" iyy="1e-6" iyz="0" izz="1e-6"/>
+        </inertial>
+        <collision>
+        <origin xyz="0 0 0" rpy="0 0 0"/>
+        <geometry>
+            <box size="0.1 0.1 0.1"/>
+        </geometry>
+        </collision>
+        <visual>
+        <origin xyz="0 0 0" rpy="0 0 0"/>
+        <geometry>
+            <mesh filename="package://my_robot/meshes/hokuyo.dae"/>
+        </geometry>
+        </visual>
+    </link>
+    <joint name="cm_joint" type="fixed">
+        <origin xyz="0 0 0" rpy="0 0 0"/>
+        <parent link="robot_footprint"/>
+        <child link="crossbar_main"/>
+    </joint>
+    <joint name="ctf_joint" type="fixed">
+        <origin xyz="0 0.275 0" rpy="0 0 0"/>
+        <parent link="robot_footprint"/>
+        <child link="crossbar_trans_forward"/>
+    </joint>
+    <joint name="ctc_joint" type="fixed">
+        <origin xyz="0 0.1 0" rpy="0 0 0"/>
+        <parent link="robot_footprint"/>
+        <child link="crossbar_trans_center"/>
+    </joint>
+    <joint name="tail_joint" type="fixed">
+        <origin xyz="0 -0.25 0.05" rpy="0 0 0"/>
+        <parent link="robot_footprint"/>
+        <child link="tail"/>
+    </joint>
+    <joint type="continuous" name="left_wheel_hinge">
+        <origin xyz="0.225 0 0" rpy="0 0 0"/>
+        <child link="left_wheel"/>
+        <parent link="crossbar_trans_center"/>
+        <axis xyz="0 1 0" rpy="0 0 0"/>
+        <limit effort="10000" velocity="1000"/>
+        <dynamics damping="1.0" friction="1.0"/>
+    </joint>
+    <joint type="continuous" name="right_wheel_hinge">
+        <origin xyz="-0.225 0 0" rpy="0 0 0"/>
+        <child link="right_wheel"/>
+        <parent link="crossbar_trans_center"/>
+        <axis xyz="0 1 0" rpy="0 0 0"/>
+        <limit effort="10000" velocity="1000"/>
+        <dynamics damping="1.0" friction="1.0"/>
+    </joint>
+    <joint type="fixed" name="camera_joint">
+        <origin xyz="0 0.15 0.1" rpy="0 0 0"/>
+        <axis xyz="0 1 0"/>
+        <parent link="tail"/>
+        <child link="camera"/>
+    </joint>
+    <joint type="fixed" name="hokuyo_joint">
+        <origin xyz="0 0.25 0.05" rpy="0 0 0"/>
+        <axis xyz="0 1 0"/>
+        <parent link="crossbar_main"/>
+        <child link="hokuyo"/>
+    </joint>
+    <gazebo reference="crossbar_main">
+        <material>Gazebo/Red</material>
+    </gazebo>
+    <gazebo reference="crossbar_trans_forward">
+        <material>Gazebo/Red</material>
+    </gazebo>
+    <gazebo reference="crossbar_trans_center">
+        <material>Gazebo/Red</material>
+    </gazebo>
+    <gazebo reference="tail">
+        <material>Gazebo/Red</material>
+    </gazebo>
+    <gazebo reference="left_wheel">
+        <material>Gazebo/Black</material>
+    </gazebo>
+    <gazebo reference="right_wheel">
+        <material>Gazebo/Black</material>
+    </gazebo>
+    <gazebo reference="camera">
+        <material>Gazebo/Blue</material>
+    </gazebo>
 </robot>

Commit message: RViz Integration

File: my_robot/urdf/my_robot.xacro (robot description, xacro)
@@ -153,20 +153,20 @@
     <link name="camera">
         <inertial>
-        <mass value="0.1"/>
-        <origin xyz="0 0 0" rpy="0 0 0"/>
-        <box_inertia sizeX="0.05" sizeY="0.05" sizeZ="0.05" mass="0.1"/>
-        <inertia ixx="1e-6" ixy="0" ixz="0" iyy="1e-6" iyz="0" izz="1e-6"/>
-        </inertial>
-        <collision>
-        <origin xyz="0 0 0" rpy="1.5707 0 0"/>
-        <geometry>
-            <cylinder radius="0.025" length="0.05"/>
-        </geometry>
-        </collision>
-        <visual>
-        <origin xyz="0 0 0" rpy="1.5707 0 0"/>
-        <geometry>
-            <cylinder radius="0.025" length="0.05"/>
-        </geometry>
+            <mass value="0.1"/>
+            <origin xyz="0 0 0" rpy="0 0 0"/>
+            <box_inertia sizeX="0.05" sizeY="0.05" sizeZ="0.05" mass="0.1"/>
+            <inertia ixx="1e-6" ixy="0" ixz="0" iyy="1e-6" iyz="0" izz="1e-6"/>
+        </inertial>
+        <collision>
+            <origin xyz="0 0 0" rpy="1.5707 0 0"/>
+            <geometry>
+                <cylinder radius="0.025" length="0.05"/>
+            </geometry>
+        </collision>
+        <visual>
+            <origin xyz="0 0 0" rpy="1.5707 0 0"/>
+            <geometry>
+                <cylinder radius="0.025" length="0.05"/>
+            </geometry>
         </visual>
     </link>
@@ -174,8 +174,8 @@
         <inertial>
         <mass value="1e-1"/>
-        <origin xyz="0 0 0" rpy="0 0 0"/>
-        <box_inertia sizeX="0.05" sizeY="0.05" sizeZ="0.05" mass="0.1"/>
-        <inertia ixx="1e-6" ixy="0" ixz="0" iyy="1e-6" iyz="0" izz="1e-6"/>
-        </inertial>
+            <origin xyz="0 0 0" rpy="0 0 0"/>
+            <box_inertia sizeX="0.05" sizeY="0.05" sizeZ="0.05" mass="0.1"/>
+            <inertia ixx="1e-6" ixy="0" ixz="0" iyy="1e-6" iyz="0" izz="1e-6"/>
+            </inertial>
         <collision>
         <origin xyz="0 0 0" rpy="0 0 0"/>
@@ -228,5 +228,5 @@
     </joint>
     <joint type="fixed" name="camera_joint">
-        <origin xyz="0 0.15 0.1" rpy="0 0 0"/>
+        <origin xyz="0 0.15 0.1" rpy="0 0 1.5707"/>
         <axis xyz="0 1 0"/>
         <parent link="tail"/>

Commit message: Setting up ball chaser. Robot model is fixed.

File: my_robot/urdf/my_robot.xacro (robot description, xacro)
@@ -215,5 +215,5 @@
         <child link="left_wheel"/>
         <parent link="crossbar_trans_center"/>
-        <axis xyz="0 1 0" rpy="0 0 0"/>
+        <axis xyz="-1 0 0" rpy="0 0 0"/>
         <limit effort="10000" velocity="1000"/>
         <dynamics damping="1.0" friction="1.0"/>
@@ -223,5 +223,5 @@
         <child link="right_wheel"/>
         <parent link="crossbar_trans_center"/>
-        <axis xyz="0 1 0" rpy="0 0 0"/>
+        <axis xyz="-1 0 0" rpy="0 0 0"/>
         <limit effort="10000" velocity="1000"/>
         <dynamics damping="1.0" friction="1.0"/>

Commit message: Camera is rotated.

File: my_robot/urdf/my_robot.xacro (robot description, xacro)
@@ -159,5 +159,5 @@
         </inertial>
         <collision>
-            <origin xyz="0 0 0" rpy="1.5707 0 0"/>
+            <origin xyz="0 0 0" rpy="0 1.5707 0"/>
             <geometry>
                 <cylinder radius="0.025" length="0.05"/>
@@ -165,5 +165,5 @@
         </collision>
         <visual>
-            <origin xyz="0 0 0" rpy="1.5707 0 0"/>
+            <origin xyz="0 0 0" rpy="0 1.5707 0"/>
             <geometry>
                 <cylinder radius="0.025" length="0.05"/>

Commit message: Robot goes straght forward without deviation. robot_footprint is used only for chassis. Tail is made liter.

File: my_robot/urdf/my_robot.xacro (robot description, xacro)
@@ -4,5 +4,4 @@
     <link name="robot_footprint"></link>
     <link name="crossbar_main">
-        <pose>0 0 0.1 0 0 0</pose>
         <inertial>
             <mass value="1.0"/>
@@ -23,5 +22,5 @@
             <origin xyz="0 0 0" rpy=" 0 0 0"/>
             <geometry>
-                <box size="0.1 0.5 0.05"/>
+                <box size="0.1 0.5 0.049"/>
             </geometry>
         </visual>
@@ -29,5 +28,5 @@
             <origin xyz="0 -0.25 -0.05" rpy=" 0 0 0"/>
             <geometry>
-                <sphere radius="0.05"/>
+                <sphere radius="0.049"/>
             </geometry>
         </collision>
@@ -35,8 +34,30 @@
             <origin xyz="0 -0.25 -0.05" rpy=" 0 0 0"/>
             <geometry>
+                <sphere radius="0.049"/>
+            </geometry>
+        </visual>
+        <collision name='caster_collision_fw'>
+            <origin xyz="0 0.24 -0.05" rpy=" 0 0 0"/>
+            <geometry>
+                <sphere radius="0.049"/>
+            </geometry>
+        </collision>
+        <visual name='caster_visual_fw'>
+            <origin xyz="0 0.24 -0.05" rpy=" 0 0 0"/>
+            <geometry>
                 <sphere radius="0.05"/>
             </geometry>
         </visual>
     </link>
+    <joint name="ctc_joint" type="fixed">
+        <origin xyz="0 0.1 0" rpy="0 0 0"/>
+        <parent link="robot_footprint"/>
+        <child link="crossbar_trans_center"/>
+    </joint>
+    <joint name="cm_joint" type="fixed">
+        <origin xyz="0 0 0" rpy="0 0 0"/>
+        <parent link="crossbar_trans_center"/>
+        <child link="crossbar_main"/>
+    </joint>
     <link name="crossbar_trans_forward">
         <pose>0 0 0.1 0 0 0</pose>
@@ -63,6 +84,10 @@
         </visual>
     </link>
+    <joint name="ctf_joint" type="fixed">
+        <origin xyz="0 0.275 0" rpy="0 0 0"/>
+        <parent link="robot_footprint"/>
+        <child link="crossbar_trans_forward"/>
+    </joint>
     <link name="crossbar_trans_center">
-        <pose>0 0 0.1 0 0 0</pose>
         <inertial>
             <mass value="0.5"/>
@@ -90,10 +115,10 @@
         <pose>0 0 0.1 0 0 0</pose>
         <inertial>
-            <mass value="0.5"/>
-            <origin xyz="0.0 0 0" rpy=" 0 0 0"/>
-            <inertia
-                ixx="0.1" ixy="0" ixz="0"
-                iyy="0.1" iyz="0"
-                izz="0.1"
+            <mass value="0.25"/>
+            <origin xyz="0.0 0 0" rpy=" 0 0 0"/>
+            <inertia
+                ixx="0.01" ixy="0" ixz="0"
+                iyy="0.01" iyz="0"
+                izz="0.01"
             />
         </inertial>
@@ -111,4 +136,9 @@
         </visual>
     </link>
+    <joint name="tail_joint" type="fixed">
+        <origin xyz="0 -0.25 0.05" rpy="0 0 0"/>
+        <parent link="crossbar_main"/>
+        <child link="tail"/>
+    </joint>
     <link name="left_wheel">
         <pose>0 0 0.1 0 0 0</pose>
@@ -131,4 +161,12 @@
         </visual>
     </link>
+    <joint type="continuous" name="left_wheel_hinge">
+        <origin xyz="-0.225 0 0" rpy="0 0 0"/>
+        <child link="left_wheel"/>
+        <parent link="crossbar_trans_center"/>
+        <axis xyz="-1 0 0" rpy="0 0 0"/>
+        <limit effort="10000" velocity="1000"/>
+        <dynamics damping="1.0" friction="1.0"/>
+    </joint>
     <link name="right_wheel">
         <pose>0 0 0.1 0 0 0</pose>
@@ -151,4 +189,12 @@
         </visual>
     </link>
+    <joint type="continuous" name="right_wheel_hinge">
+        <origin xyz="0.225 0 0" rpy="0 0 0"/>
+        <child link="right_wheel"/>
+        <parent link="crossbar_trans_center"/>
+        <axis xyz="-1 0 0" rpy="0 0 0"/>
+        <limit effort="10000" velocity="1000"/>
+        <dynamics damping="1.0" friction="1.0"/>
+    </joint>
     <link name="camera">
         <inertial>
@@ -171,4 +217,10 @@
         </visual>
     </link>
+    <joint type="fixed" name="camera_joint">
+        <origin xyz="0 0.15 0.1" rpy="0 0 1.5707"/>
+        <axis xyz="0 1 0"/>
+        <parent link="tail"/>
+        <child link="camera"/>
+    </joint>
     <link name="hokuyo">
         <inertial>
@@ -191,47 +243,5 @@
         </visual>
     </link>
-    <joint name="cm_joint" type="fixed">
-        <origin xyz="0 0 0" rpy="0 0 0"/>
-        <parent link="robot_footprint"/>
-        <child link="crossbar_main"/>
-    </joint>
-    <joint name="ctf_joint" type="fixed">
-        <origin xyz="0 0.275 0" rpy="0 0 0"/>
-        <parent link="robot_footprint"/>
-        <child link="crossbar_trans_forward"/>
-    </joint>
-    <joint name="ctc_joint" type="fixed">
-        <origin xyz="0 0.1 0" rpy="0 0 0"/>
-        <parent link="robot_footprint"/>
-        <child link="crossbar_trans_center"/>
-    </joint>
-    <joint name="tail_joint" type="fixed">
-        <origin xyz="0 -0.25 0.05" rpy="0 0 0"/>
-        <parent link="robot_footprint"/>
-        <child link="tail"/>
-    </joint>
-    <joint type="continuous" name="left_wheel_hinge">
-        <origin xyz="0.225 0 0" rpy="0 0 0"/>
-        <child link="left_wheel"/>
-        <parent link="crossbar_trans_center"/>
-        <axis xyz="-1 0 0" rpy="0 0 0"/>
-        <limit effort="10000" velocity="1000"/>
-        <dynamics damping="1.0" friction="1.0"/>
-    </joint>
-    <joint type="continuous" name="right_wheel_hinge">
-        <origin xyz="-0.225 0 0" rpy="0 0 0"/>
-        <child link="right_wheel"/>
-        <parent link="crossbar_trans_center"/>
-        <axis xyz="-1 0 0" rpy="0 0 0"/>
-        <limit effort="10000" velocity="1000"/>
-        <dynamics damping="1.0" friction="1.0"/>
-    </joint>
-    <joint type="fixed" name="camera_joint">
-        <origin xyz="0 0.15 0.1" rpy="0 0 1.5707"/>
-        <axis xyz="0 1 0"/>
-        <parent link="tail"/>
-        <child link="camera"/>
-    </joint>
-    <joint type="fixed" name="hokuyo_joint">
+     <joint type="fixed" name="hokuyo_joint">
         <origin xyz="0 0.25 0.05" rpy="0 0 0"/>
         <axis xyz="0 1 0"/>
