Commit message: Stable is done.

File: my_robot/urdf/my_robot.xacro (robot description, xacro)
@@ -5,10 +5,10 @@
     <link name="crossbar_main">
         <inertial>
-            <mass value="1.0"/>
-            <origin xyz="0.0 0 0" rpy=" 0 0 0"/>
-            <inertia
-                ixx="0.1" ixy="0" ixz="0"
-                iyy="0.1" iyz="0"
-                izz="0.1"
+            <mass value="0.5"/>
+            <origin xyz="0.0 0 0" rpy=" 0 0 0"/>
+            <inertia
+                ixx="1e-2" ixy="0" ixz="0"
+                iyy="1e-2" iyz="0"
+                izz="1e-2"
             />
         </inertial>
@@ -44,5 +44,5 @@
         </collision>
         <visual name='caster_visual_fw'>
-            <origin xyz="0 0.24 -0.05" rpy=" 0 0 0"/>
+            <origin xyz="0 0.20 -0.05" rpy=" 0 0 0"/>
             <geometry>
                 <sphere radius="0.05"/>
@@ -61,12 +61,11 @@
     </joint>
     <link name="crossbar_trans_forward">
-        <pose>0 0 0.1 0 0 0</pose>
-        <inertial>
-            <mass value="0.5"/>
-            <origin xyz="0.0 0 0" rpy=" 0 0 0"/>
-            <inertia
-                ixx="0.1" ixy="0" ixz="0"
-                iyy="0.1" iyz="0"
-                izz="0.1"
+        <inertial>
+            <mass value="0.5"/>
+            <origin xyz="0.0 0 0" rpy=" 0 0 0"/>
+            <inertia
+                ixx="1e-2" ixy="0" ixz="0"
+                iyy="1e-2" iyz="0"
+                izz="1e-2"
             />
         </inertial>
@@ -91,10 +90,10 @@
     <link name="crossbar_trans_center">
         <inertial>
-            <mass value="0.5"/>
-            <origin xyz="0.0 0 0" rpy=" 0 0 0"/>
-            <inertia
-                ixx="0.1" ixy="0" ixz="0"
-                iyy="0.1" iyz="0"
-                izz="0.1"
+            <mass value="5"/>
+            <origin xyz="0.0 0 0" rpy=" 0 0 0"/>
+            <inertia
+                ixx="1e-2" ixy="0" ixz="0"
+                iyy="1e-2" iyz="0"
+                izz="1e-2"
             />
         </inertial>
@@ -113,5 +112,4 @@
     </link>
     <link name="tail">
-        <pose>0 0 0.1 0 0 0</pose>
         <inertial>
             <mass value="0.25"/>
@@ -142,14 +140,13 @@
     </joint>
     <link name="left_wheel">
-        <pose>0 0 0.1 0 0 0</pose>
-        <collision>
-            <geometry>
-                <cylinder radius="0.1" length="0.05"/>
-            </geometry>
-            <origin xyz="0 0 0" rpy="0 1.5707 0"/>
-        </collision>
-        <inertial>
-            <origin xyz="0 0 0" rpy="0 1.5707 0"/>
-            <mass value="0.1"/>
+        <collision>
+            <geometry>
+                <cylinder radius="0.1" length="0.05"/>
+            </geometry>
+            <origin xyz="0 0 0" rpy="0 1.5707 0"/>
+        </collision>
+        <inertial>
+            <origin xyz="0 0 0" rpy="0 1.5707 0"/>
+            <mass value="0.5"/>
             <inertia ixx="0.1" ixy="0" ixz="0"  iyy="0.1" iyz="0" izz="0.1"/>
         </inertial>
@@ -170,14 +167,13 @@
     </joint>
     <link name="right_wheel">
-        <pose>0 0 0.1 0 0 0</pose>
-        <collision>
-            <geometry>
-                <cylinder radius="0.1" length="0.05"/>
-            </geometry>
-            <origin xyz="0 0 0" rpy="0 1.5707 0"/>
-        </collision>
-        <inertial>
-            <origin xyz="0 0 0" rpy="0 1.5707 0"/>
-            <mass value="0.1"/>
+        <collision>
+            <geometry>
+                <cylinder radius="0.1" length="0.05"/>
+            </geometry>
+            <origin xyz="0 0 0" rpy="0 1.5707 0"/>
+        </collision>
+        <inertial>
+            <origin xyz="0 0 0" rpy="0 1.5707 0"/>
+            <mass value="0.5"/>
             <inertia ixx="0.1" ixy="0" ixz="0"  iyy="0.1" iyz="0" izz="0.1"/>
         </inertial>

Commit message: feat: Move the lidar to the tail

File: my_robot/urdf/my_robot.xacro (robot description, xacro)
@@ -138,4 +138,33 @@
         <parent link="crossbar_main"/>
         <child link="tail"/>
+    </joint>
+    <link name="small_tail">
+        <inertial>
+            <mass value="0.001"/>
+            <origin xyz="0.0 0 0" rpy=" 0 0 0"/>
+            <inertia
+                ixx="0.01" ixy="0" ixz="0"
+                iyy="0.01" iyz="0"
+                izz="0.01"
+            />
+        </inertial>
+        <collision name='small_tail_collision'>
+            <origin xyz="0 0 0" rpy=" 0 0 0"/>
+            <geometry>
+                <cylinder radius="0.05" length="0.05"/>
+            </geometry>
+        </collision>
+        <visual name='small_tail_visual'>
+            <origin xyz="0 0 0" rpy=" 0 0 0"/>
+            <geometry>
+                <cylinder radius="0.05" length="0.05"/>
+            </geometry>
+        </visual>
+    </link>
+    <joint type="fixed" name="small_tail_joint">
+        <origin xyz="0 -0.1 0.1" rpy="0 0 1.5707"/>
+        <axis xyz="0 1 0"/>
+        <parent link="tail"/>
+        <child link="small_tail"/>
     </joint>
     <link name="left_wheel">
@@ -239,8 +268,8 @@
         </visual>
     </link>
-     <joint type="fixed" name="hokuyo_joint">
-        <origin xyz="0 0.25 0.05" rpy="0 0 0"/>
+    <joint type="fixed" name="hokuyo_joint">
+        <origin xyz="0 0 0.05" rpy="0 0 0"/>
         <axis xyz="0 1 0"/>
-        <parent link="crossbar_main"/>
+        <parent link="small_tail"/>
         <child link="hokuyo"/>
     </joint>
@@ -255,4 +284,7 @@
     </gazebo>
     <gazebo reference="tail">
+        <material>Gazebo/Red</material>
+    </gazebo>
+    <gazebo reference="small__tail">
         <material>Gazebo/Red</material>
     </gazebo>

Commit message: feat: Add optical camera link

File: my_robot/urdf/my_robot.xacro (robot description, xacro)
@@ -247,4 +247,11 @@
         <parent link="tail"/>
         <child link="camera"/>
+    </joint>
+    <link name="camera_link_optical">
+    </link>
+    <joint name="camera_optical_joint" type="fixed">
+        <origin xyz="0 0 0" rpy="-1.5707 0 -1.5707"/>
+        <parent link="camera"/>
+        <child link="camera_link_optical"/>
     </joint>
     <link name="hokuyo">

Commit message: bug: Change optical camera position

File: my_robot/urdf/my_robot.xacro (robot description, xacro)
@@ -251,5 +251,5 @@
     </link>
     <joint name="camera_optical_joint" type="fixed">
-        <origin xyz="0 0 0" rpy="-1.5707 0 -1.5707"/>
+        <origin xyz="0 0 0" rpy="1.5707 3.1416 0"/>
         <parent link="camera"/>
         <child link="camera_link_optical"/>
